File: src/hardware/CyDAQ/Filter Board/Filter Board.brd (EAGLE design)
At the start: 160.9 x 110.9 mm, 213 parts, among them J1 DCJ0202, J10 Vout_HEADER, J11 5V0_SENSOR, J12 3V3_SENSOR, J13 1V8_SENSOR, J14 BRKOUT_JD, J15 BRKOUT_JC, J16 BRKOUT_JB, J17 BRKOUT_JF, J18 5V0_CONN, J19 3V3_CONN, J2 ZYBO_JF, J20 1V8_CONN, J3 ZYBO_JE, J4 ZYBO_JD, J5 ZYBO_JC, J6 ZYBO_JB, J7 A_XADC, J8 SJ1-3523N, J9 Vin_HEADER, U1 TPS54531DDARDDA8_3P1X2P4-L, U10 CD74HCT4051, U11 CD74HCT4051, U12 OPA4197, U13 OPA4197, U14 OPA4197, U15 OPA4197, U16 OPA4197, U17 CD74HCT4053, U18 CD74HCT4051, U19 OPA2197, U2 VS-50WQ04FNPBFDPAK-L, U3 TPS56339, U4 TPS56339, U5 LM43601PWPR, U6 X9258_A, U7 X925_B, U8 X9258_C, U9 X9258_D

Commit message: Finished routing main filter area
Parts:
- removed TP1, TP2: JF7, testpad:P1-17
- added J21: BRKOUT_JD, Connectors:FEMALE_HEADER-2X6
- moved C27 204.7 mm to (62.2, 67.3), turned to 270 degrees
- moved R40 198.2 mm to (52.8, 58.7)
- moved R39 197.9 mm to (54.2, 63.0), turned to 270 degrees
- moved C34 197.5 mm to (57.0, 63.0)
- moved C31 196.8 mm to (51.4, 63.0), turned to 270 degrees
- moved R46 196.4 mm to (59.8, 63.0), turned to 270 degrees
- moved C35 193.5 mm to (58.4, 58.7), turned to 270 degrees
- moved R43 192.4 mm to (55.6, 58.7)
- moved U10 191.1 mm to (69.3, 65.3), turned to 270 degrees
- moved C24 177.6 mm to (76.5, 62.5)
- moved R41 175.1 mm to (93.5, 64.0)
- moved R42 175.1 mm to (93.5, 60.7)
- moved C22 175.0 mm to (52.8, 69.6), turned to 90 degrees
- moved C25 175.0 mm to (62.2, 55.6)
- moved C28 175.0 mm to (76.5, 52.1)
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Connections:
- net 3V3: now also J21.1, J21.2
- net BP2_IN: now also U10.5; no longer U10.1
- net BP6_IN: now also U10.1; no longer U10.5
- net BP6_OUT: now also U11.12; no longer U11.5
- net GND: now also J21.3, J21.4
- net HP1_IN: now also U10.12; no longer U10.15
- net JF7: no longer TP2.TP
- net JF8: no longer TP1.TP
- net LP1_IN: now also U10.15; no longer U10.12
- net LP1_OUT: now also U11.5; no longer U11.12
- net XADC_J14: now also J21.5
- net XADC_J16: now also J21.7
- net XADC_K14: now also J21.6
- net XADC_K16: now also J21.8
- net XADC_L14: now also J21.10
- net XADC_L15: now also J21.9
Routing:
- net FILTER_OUT_BUFF: track 1.27 -> 144.7 mm, vias 0 -> 2
- net BP6_IN: track 0.00 -> 70.9 mm, vias 0 -> 2
- net LP2_OUT1: track 3.51 -> 73.1 mm
- net !HP!/LP_TOGGLE: track 2.54 -> 66.5 mm
- net HP2_OUT1: track 24.7 -> 86.4 mm
- net BP6_OUT: track 1.27 -> 37.9 mm, vias 0 -> 2
- net FILTER_IN: track 0.00 -> 29.8 mm
- net LP1_IN: track 1.27 -> 29.5 mm
- net N$23: track 2.54 -> 30.6 mm, vias 0 -> 2
- net HP/LP2_IN1: track 0.00 -> 24.8 mm
- net BP2_IN: track 0.00 -> 21.7 mm
- net NOTCH_IN: track 3.20 -> 18.6 mm
- net NOTCH_OUT: track 5.28 -> 18.2 mm
- net N$73: track 0.00 -> 12.0 mm
- net XADC_N15: track 0.00 -> 11.0 mm
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Other:
- board text added: "Set ref plane pullback"
- board text removed: "Notch Filter"
