File: src/hardware/CyDAQ/CyDAQ/Filter Board.sch (EAGLE design)
At the start: 214 parts, among them J1 DCJ0202, J10 Vout_HEADER, J11 5V0_SENSOR, J12 3V3_SENSOR, J13 1V8_SENSOR, J14 BRKOUT_JD, J15 BRKOUT_JC, J16 BRKOUT_JB, J17 BRKOUT_JF, J18 5V0_CONN, J19 3V3_CONN, J2 ZYBO_JF, J20 1V8_CONN, J21 BRKOUT_JD, J22 ZYBO_Power, J3 ZYBO_JE, J4 ZYBO_JD, J5 ZYBO_JC, J6 ZYBO_JB, J7 A_XADC, J8 SJ1-3523N, J9 Vin_HEADER, U1 TPS54531DDARDDA8_3P1X2P4-L, U10 CD74HCT4051, U11 CD74HCT4051, U12 OPA4197, U13 OPA4197, U14 OPA4197, U15 OPA4197, U16 OPA4197, U17 CD74HCT4053, U18 CD74HCT4051, U19 OPA2197, U3 TPS56339, U4 TPS56339, U5 LM43601PWPR, U6 X9258_A, U7 X925_B, U8 X9258_C, U9 X9258_D

Commit message: Adding Sam's redesgined PMICs
Parts:
- removed -5V: TPPAD1-13, testpad:TPPAD1-13
- added -5V0: TPPAD1-13, testpad:TPPAD1-13
Connections:
- net N$15 renamed FB
- net N$16 renamed SW
- net N$19 renamed BOOT
- net N$20 renamed PGOOD
- net +5V0: no longer C16.1, C17.1, U5.EN, U5.VIN, U5.VIN_2
- net -5V0: now also -5V0.TP; no longer -5V.TP
- net 12V0: now also C16.1, C17.1, U5.EN, U5.VIN, U5.VIN_2
Other:
- moved on the sheet: C15, C16, C17, C18, C19, C20, C21, G4, L4, R10, R11, R12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
